File: edl_schematic/small_one/small.brd (EAGLE design)
At the start: 161.3 x 119 mm, 50 parts, among them IC1 TL084D, IC11 TL084D, IC18 TL084D, IC19 TL084D, IC23 TL084D, IC3 TL084D, U3 TLV5610_DW_20, U4 MAX395EWG

Commit message: small one completed
i guess
Parts:
- added JP5, JP6: (no value), jumper:JP6Q
- added JP7: (no value), jumper:JP2Q
- moved U4 16.3 mm to (41.9, 22.9)
Connections:
- removed net +12V: IC1.4, IC11.4, IC18.4, IC19.4, IC23.4, IC3.4
- removed net +3.3V: R116.1, R122.1, R31.1, R67.1
- removed net -12V: IC1.11, IC11.11, IC18.11, IC19.11, IC23.11, IC3.11
- new net +5V: IC1.4, IC11.4, IC18.4, IC19.4, IC23.4, IC3.4, JP7.1
- new net -5V: IC1.11, IC11.11, IC18.11, IC19.11, IC23.11, IC3.11, JP7.3
- new net A11Q: JP5.11, U4.7
- new net FS: JP1.4, U3.4
- new net LDAC: JP1.6, U3.18
- new net MODE: JP1.8, U3.17
- new net PRE: JP1.2, U3.5
- new net REF: JP1.10, U3.16
- net 3V3: now also JP5.4, JP6.10, JP7.2, R116.1, R122.1, R31.1, R67.1
- net A1P: now also JP5.9
- net A1Q: no longer U4.7
- net A3P: now also JP5.10
- net A3Q: now also JP5.12
- net A5P: now also JP5.1
- net A5Q: now also JP5.3
- net A7P: now also JP5.7
- net A7Q: now also JP5.5
- net B1P: now also JP6.4
- net B1Q: now also JP6.2
- net B3P: now also JP6.3
- net B3Q: now also JP6.1
- net B5P: now also JP6.5
- net B5Q: now also JP6.7
- net B7P: now also JP6.11
- net B7Q: now also JP6.9
- net CHAN_E11: now also JP1.14; no longer JP1.8
- net CHAN_F11: now also JP1.16; no longer JP1.10
- net CS_SW: now also JP6.12
- net GND: now also JP5.8, JP6.6, JP7.4
- net SPI_CLK_SW: now also JP5.2
- net SPI_MOSI_SW: now also JP5.6
- net TO_NEXT1: now also JP6.8
Routing:
- net +5V: track 0.00 -> 468.7 mm, vias 0 -> 7
- net 3V3: track 0.00 -> 416.2 mm, vias 0 -> 7
- net -5V: track 0.00 -> 380.5 mm, vias 0 -> 6
- net GND: track 14.6 -> 104.9 mm, vias 0 -> 2
- net REF: track 0.00 -> 71.4 mm
- net MODE: track 0.00 -> 65.5 mm
- net LDAC: track 0.00 -> 59.7 mm
- net FS: track 0.00 -> 49.3 mm
- net PRE: track 0.00 -> 36.3 mm
- net N$109: track 7.41 -> 36.8 mm, vias 0 -> 2
- net A5P: track 0.00 -> 27.9 mm
- net CS_SW: track 0.00 -> 26.9 mm
- net N$115: track 7.93 -> 33.6 mm, vias 0 -> 2
- net B7P: track 0.00 -> 25.4 mm
- net A5Q: track 0.00 -> 24.0 mm
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- added copper zone on layer 1, net GND
Other:
- board size 161.3 x 119 mm -> 160 x 137.3 mm

Commit message: small board done
Parts:
- moved R26 4.83 mm to (138.2, -7.62)
- moved R62 3.56 mm to (136.9, 30.5)
- moved R65 3.06 mm to (100.6, 38.6)
- moved R69 2.55 mm to (106.7, 30.7)
- moved R115 2.03 mm to (55.4, 76.2)
- moved IC1 1.78 mm to (117.3, 67.3)
- moved IC19 0.80 mm to (61.5, 58.2)
Routing:
- net 3V3: track 416.2 -> 500.7 mm
- net GND: track 104.9 -> 143.4 mm, vias 2 -> 6
- net -5V: track 380.5 -> 395.1 mm
- net N$36: track 10.2 -> 17.6 mm
- net N$70: track 36.6 -> 42.4 mm
- net N$68: track 13.8 -> 18.8 mm
- net +5V: track 468.7 -> 473.6 mm
- net N$74: track 29.2 -> 34.1 mm
- net VIN11: track 114.5 -> 109.6 mm
- net VIN22: track 58.3 -> 54.7 mm
- net ADC_IN2: track 55.7 -> 58.5 mm
- net N$71: track 59.6 -> 57.3 mm
- net CS_SW: track 26.9 -> 29.1 mm
- net N$110: track 29.4 -> 27.4 mm
- net N$109: track 36.8 -> 38.9 mm
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