File: edl_schematic/final_schematic.brd (EAGLE design)
At the start: 329.6 x 243.8 mm, 303 parts, among them CON1 UBC05V128-B0C04D, IC1 FT232RL, IC14 TL084D, IC15 TL084D, IC16 TL084D, IC17 TL084D, IC18 TL084D, IC19 TL084D, IC20 TL084D, IC21 TL084D, IC22 TL084D, IC23 TL084D, IC24 TL084D, IC25 TL084D, IC26 TL084D, IC27 TL084D, IC28 TL084D, IC29 TL084D, IC3 TL084D, IC30 TL084D, IC4 TPS77333, IC5 TL084D, IC6 7812TV, Q1 BC558B, U1 TMS320F28069_PN_80, U3 TLV5610_DW_20, U4 MAX395EWG, U6 MAX395EWG, U7 MAX395EWG

Commit message: final touches thursday
Parts:
- removed F1: 500mA, rcl:L1812
- added R24: (no value), adafruit:0207/7
- moved R23 8.68 mm to (50.1, 34.3), flipped to the bottom, turned to 270 degrees
Connections:
- removed net CTS: IC1.11
- removed net DCD: IC1.10
- removed net DSR: IC1.9
- removed net N$17: C3.1, F2.1
- removed net RI: IC1.6
- removed net XUSB: CON1.1, F1.2
- new net DGND: C1.2, C10.2, C11.1, C12.1, C13.1, C14.2, C15.2, C16.2, C17.1, C18.1, C19.1, C2.1, C20.2, C21.2, C22.1, C3.2, C4.2, C43.1, C5.2, C7.2, C8.2, C9.2, CON1.5, IC1.18, IC1.21, IC1.25, IC1.26, IC1.7, JP4.11, Q1.C, R10.1, R17.1, R24.1, R8.1, S2.P$1, S2.P$2, SV2.10, SV2.12, SV2.4, SV2.8, U1.13, U1.21, U1.28, U1.3, U1.38, U1.50, U1.64, U1.71, U1.73, U3.1, U3.10, U3.18
- new net VBUS_ORG: C3.1, CON1.1, F2.1
- net GND: now also R24.2; no longer C1.2, C10.2, C11.1, C12.1, C13.1, C14.2, C15.2, C16.2, C17.1, C18.1, C19.1, C2.1, C20.2, C21.2, C22.1, C3.2, C4.2, C43.1, C5.2, C7.2, C8.2, C9.2, CON1.5, IC1.18, IC1.21, IC1.25, IC1.26, IC1.7, JP4.11, Q1.C, R10.1, R17.1, R8.1, S2.P$1, S2.P$2, SV2.10, SV2.12, SV2.4, SV2.8, U1.13, U1.21, U1.28, U1.3, U1.38, U1.50, U1.64, U1.71, U1.73, U3.1, U3.10, U3.18
- net VBUS: no longer F1.1
Routing:
- net DGND: track 0.00 -> 250.3 mm, vias 0 -> 22
- net GND: track 353.4 -> 176.8 mm, vias 41 -> 24
- net VBUS_ORG: track 0.00 -> 61.1 mm, vias 0 -> 1
- net VBUS: track 94.4 -> 45.0 mm
- net N$16: track 2.98 -> 14.7 mm, vias 0 -> 1
- net XUSB: track 11.5 -> 0.00 mm
- net +12V: track 1894.5 -> 1888.5 mm
- net N$17: track 4.78 -> 0.00 mm
- net 3V3: track 1595.4 -> 1599.3 mm, vias 35 -> 34
- net N$23: track 34.9 -> 36.5 mm
- net -12V: track 1701.5 -> 1702.5 mm
- net VIN-: track 8.12 -> 8.91 mm
- net N$30: track 15.6 -> 14.9 mm
- net SPI_CS: track 62.3 -> 61.6 mm
- net SPI_MOSI: track 42.6 -> 42.1 mm
- added copper zone on layer 1, net DGND
- added copper zone on layer 16, net DGND
Other:
- board size 329.6 x 243.8 mm -> 329.5 x 243.7 mm
- board text added: "BT002"
- board text added: "DPAC D03,D11,D13"
