File: edl_schematic/final_schematic.sch (EAGLE design)
At the start: 299 parts, among them CON1 UBC05V128-B0C04D, IC1 FT232RL, IC14 TL084D, IC15 TL084D, IC16 TL084D, IC17 TL084D, IC18 TL084D, IC19 TL084D, IC20 TL084D, IC21 TL084D, IC22 TL084D, IC23 TL084D, IC24 TL084D, IC25 TL084D, IC26 TL084D, IC27 TL084D, IC28 TL084D, IC29 TL084D, IC3 TL084D, IC30 TL084D, IC4 TPS77333, IC5 TL084D, IC6 7812TV, Q1 BC558B, U1 TMS320F28069_PN_80, U3 TLV5610_DW_20, U4 MAX395EWG, U6 MAX395EWG, U7 MAX395EWG

Commit message: some small changes
written in my EDL book
Parts:
- added F2: 500mA, SparkFun:PTCSMD
- added R21, R22, R23: (no value), rcl:R-US_R1206
- renumbered D2 to D3
Connections:
- new net N$14: JP2.1, R4.2
- new net N$15: C20.1, R21.2, U1.X1, Y1.2
- new net N$16: R23.1, U1.VDD3VFL
- new net N$17: C3.1, F2.1
- net 3V3: now also R22.2, R23.2; no longer C7.1, U1.VDD3VFL, U1.VDDA
- net N$1: now also C7.1, R22.1, U1.VDDA; no longer C20.1, U1.X1, Y1.2
- net N$18: now also R21.1
- net N$23: now also D3.A; no longer D3.C
- net VBUS: now also F2.2; no longer C3.1, R4.2
- net VIN-: now also D3.C; no longer D3.A
Other:
- moved on the sheet: C20, C21, Y1

Commit message: TXD connection changed
Connections:
- net TXD: now also U1.GPIO28/SCIRXDA/SDAA/!TZ2; no longer U1.GPIO7/EPWM4B/SCIRXDA/ECAP2
Changed lines of the file:
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@@
 </segment>
 <segment>
-<pinref part="U1" gate="A" pin="GPIO7/EPWM4B/SCIRXDA/ECAP2"/>
-<wire x1="424.18" y1="5.08" x2="431.8" y2="5.08" width="0.1524" layer="91"/>
-<label x="431.8" y="5.08" size="1.778" layer="95" xref="yes"/>
+<pinref part="U1" gate="A" pin="GPIO28/SCIRXDA/SDAA/!TZ2"/>
+<wire x1="246.38" y1="-5.08" x2="246.38" y2="-10.16" width="0.1524" layer="91"/>
+<label x="246.38" y="-10.16" size="1.778" layer="95" rot="R180" xref="yes"/>
 </segment>
 </net>

Commit message: final touches thursday
Parts:
- removed F1: 500mA, rcl:L-EUL1812
- added R24: (no value), adafruit:R-US_0207/7
Connections:
- removed net CTS: IC1.!CTS
- removed net DCD: IC1.!DCD
- removed net DSR: IC1.!DSR
- removed net N$17: C3.1, F2.1
- removed net RI: IC1.!RI
- removed net XUSB: CON1.1, F1.2
- new net DGND: C1.2, C10.2, C11.1, C12.1, C13.1, C14.2, C15.2, C16.2, C17.1, C18.1, C19.1, C2.1, C20.2, C21.2, C22.1, C3.2, C4.2, C43.1, C5.2, C7.2, C8.2, C9.2, CON1.5, IC1.GND, IC1.GND@1, IC1.GND@2, IC1.GND@A, IC1.TEST, JP4.11, Q1.C, R10.1, R17.1, R24.1, R8.1, S2.0@A, S2.0@B, SV2.10, SV2.12, SV2.4, SV2.8, U1.!VREGENZ, U1.VREFLO, U1.VSS, U1.VSS_2, U1.VSS_3, U1.VSS_4, U1.VSS_5, U1.VSS_6, U1.VSS_7, U3.!LDAC, U3.AGND, U3.DGND
- new net VBUS_ORG: C3.1, CON1.1, F2.1
- net GND: now also R24.2; no longer C1.2, C10.2, C11.1, C12.1, C13.1, C14.2, C15.2, C16.2, C17.1, C18.1, C19.1, C2.1, C20.2, C21.2, C22.1, C3.2, C4.2, C43.1, C5.2, C7.2, C8.2, C9.2, CON1.5, IC1.GND, IC1.GND@1, IC1.GND@2, IC1.GND@A, IC1.TEST, JP4.11, Q1.C, R10.1, R17.1, R8.1, S2.0@A, S2.0@B, SV2.10, SV2.12, SV2.4, SV2.8, U1.!VREGENZ, U1.VREFLO, U1.VSS, U1.VSS_2, U1.VSS_3, U1.VSS_4, U1.VSS_5, U1.VSS_6, U1.VSS_7, U3.!LDAC, U3.AGND, U3.DGND
- net VBUS: no longer F1.1
Other:
- moved on the sheet: C7
