File: edl_schematic/DAC and four_var pcb/small.sch (EAGLE design)
At the start: 53 parts, among them IC1 TL084D, IC11 TL084D, IC18 TL084D, IC19 TL084D, IC23 TL084D, IC3 TL084D, U3 TLV5610_DW_20, U4 MAX395EWG

Commit message: dac,switch pcab and four variable pcb added
Parts:
- removed C1, C37: (no value), rcl:C-USC1206
- removed IC11, IC18, IC19, IC23: TL084D, linear:TL084D
- removed JP6: (no value), jumper:JP6Q
- removed R113, R114, R115, R116, R117, R118, R119, R120, R121, R122, R123, R124, R141, R145, R191, R192, R32, R62, R63, R64, R65, R66, R67, R68, R69, R70: (no value), rcl:R-US_R1206
- removed U3: TLV5610_DW_20, tlv5610a:TLV5610_DW_20
- removed U4: MAX395EWG, max395:MAX395EWG
- added C2, C3, C4, C5: (no value), rcl:C-USC1206
- added IC2: TL084D, linear:TL084D
- added R10, R11, R12, R13, R14, R15, R16, R17, R18, R19, R2, R20, R21, R22, R23, R24, R4, R5, R6, R7, R8, R9: (no value), rcl:R-US_R1206
- JP1: device jumper:JP8Q -> jumper:JP4Q
- JP2: device jumper:JP2Q -> jumper:JP4E
- JP3: device jumper:JP1Q -> jumper:JP4Q
- JP4: device jumper:JP2Q -> jumper:JP1E
- JP5: device jumper:JP6Q -> jumper:JP4E
Connections:
- removed net 3V3: JP5.4, JP6.10, JP7.2, R116.1, R122.1, R31.1, R67.1, U3.AVDD, U3.DVDD, U4.!RESET, U4.V+
- removed net A11Q: JP5.11, U4.NO1
- removed net A1P: JP5.9, U4.COM1
- removed net A1Q: C37.2, IC23A.-IN, R141.1, R145.2
- removed net A2Q: C1.2, IC1A.-IN, R1.1, R3.2
- removed net A3P: JP5.10, U4.NO0
- removed net A3Q: JP5.12, U4.COM0
- removed net A5P: JP5.1, U4.COM3
- removed net A5Q: JP5.3, U4.NO3
- removed net A7P: JP5.7, U4.NO2
- removed net A7Q: JP5.5, U4.COM2
- removed net B1P: JP6.4, U4.NO7
- removed net B1Q: JP6.2, U4.COM7
- removed net B3P: JP6.3, U4.COM6
- removed net B3Q: JP6.1, U4.NO6
- removed net B5P: JP6.5, U4.NO5
- removed net B5Q: JP6.7, U4.COM5
- removed net B7P: JP6.11, U4.COM4
- removed net B7Q: JP6.9, U4.NO4
- removed net CHAN_A: U3.OUTA
- removed net CHAN_B: U3.OUTB
- removed net CHAN_C: U3.OUTC
- removed net CHAN_D: U3.OUTD
- removed net CHAN_E: JP1.7, U3.OUTE
- removed net CHAN_E11: JP1.14, R114.1
- removed net CHAN_F: JP1.5, U3.OUTF
- removed net CHAN_F11: JP1.16, R120.1
- removed net CHAN_G: JP1.3, U3.OUTG
- removed net CHAN_H: JP1.1, U3.OUTH
- removed net CS_SW: JP6.12, U4.!CS
- removed net FS: JP1.4, U3.FS
- removed net LDAC: JP1.6, U3.!LDAC
- removed net MODE: JP1.8, U3.MODE
- removed net N$108: IC18A.-IN, R113.1, R114.2
- removed net N$109: IC18A.OUT, R113.2, R115.1
- removed net N$110: IC18B.-IN, R115.2, R116.2, R192.1
- removed net N$111: IC18D.-IN, R117.2, R118.1
- removed net N$113: IC18B.OUT, IC18D.+IN, R192.2
- removed net N$114: IC19A.-IN, R119.1, R120.2
- removed net N$115: IC19A.OUT, R119.2, R121.1
- removed net N$116: IC19B.-IN, R121.2, R122.2, R191.1
- removed net N$117: IC19D.-IN, R123.2, R124.1
- removed net N$119: IC19B.OUT, IC19D.+IN, R191.2
- removed net N$37: IC3A.OUT, R27.2, R28.1
- removed net N$39: IC3C.OUT, R29.2, R30.1
- removed net N$40: IC3B.OUT, R32.1, R34.2
- removed net N$68: IC11A.-IN, R62.2, R63.1
- removed net N$69: IC11A.OUT, R63.2, R64.1
- removed net N$70: IC11C.-IN, R64.2, R65.1
- removed net N$71: IC11C.OUT, R65.2, R66.1
- removed net N$72: IC11B.OUT, R68.1, R70.2
- removed net N$74: IC11D.-IN, R68.2, R69.1
- removed net N$75: IC11B.-IN, R66.2, R67.2, R70.1
- removed net PRE: JP1.2, U3.!PRE
- removed net REF: JP1.10, U3.REF
- removed net SPI_CLK: JP1.9, U3.SCLK
- removed net SPI_CLK_SW: JP5.2, U4.SCLK
- removed net SPI_MISO: JP1.15, U3.DOUT
- removed net SPI_MOSI: JP1.11, U3.DIN
- removed net SPI_MOSI_SW: JP5.6, U4.DIN
- removed net TO_NEXT1: JP6.8, U4.DOUT
- new net -1V65: JP4.1, R18.1, R21.1, R22.1, R24.1
- new net 1V65: JP7.2, R1.1, R12.1, R2.1, R31.1
- new net ADC_IN3: IC3B.OUT, JP5.4, R34.2
- new net ADC_IN4: IC3D.OUT, JP5.2, R33.2
- new net CHAN_F1: JP2.2, R13.1
- new net CHAN_F2: JP2.4, R15.1
- new net CHAN_F3: JP2.1, R17.1
- new net CHAN_F4: JP2.3, R23.1
- new net INTEG_IN3: IC1B.OUT, JP3.4, R20.2
- new net INTEG_IN33: JP3.5, R4.1
- new net INTEG_IN4: IC1D.OUT, JP3.8, R19.2
- new net INTEG_IN44: JP3.1, R6.1
- new net N$1: IC1A.-IN, R13.2, R14.1, R21.2
- new net N$3: IC1C.-IN, R15.2, R16.1, R22.2
- new net N$4: C5.2, IC2A.-IN, R10.2, R9.1
- new net N$5: C2.2, IC2B.-IN, R3.1, R4.2
- new net N$6: IC1D.-IN, R19.1, R23.2, R24.2
- new net N$7: IC1B.-IN, R17.2, R18.2, R20.1
- new net N$8: C3.2, IC2D.-IN, R5.1, R6.2
- new net N$9: C4.2, IC2C.-IN, R7.1, R8.2
- new net VIN3: C2.1, IC2B.OUT, JP1.8, R3.2
- new net VIN33: JP1.5, R30.1
- new net VIN4: C3.1, IC2D.OUT, JP1.4, R5.2
- new net VIN44: JP1.1, R11.1
- net +5V: now also IC2P.V+; no longer IC11P.V+, IC18P.V+, IC19P.V+, IC23P.V+
- net -5V: now also IC2P.V-; no longer IC11P.V-, IC18P.V-, IC19P.V-, IC23P.V-
- net ADC_IN1: now also IC3A.OUT, JP5.3, R27.2; no longer IC3D.OUT, JP3.1, R33.2
- net ADC_IN2: now also IC3C.OUT, JP5.1, R29.2; no longer IC11D.OUT, JP3.2, R69.2
- net GND: now also IC1B.+IN, IC1C.+IN, IC1D.+IN, IC2A.+IN, IC2B.+IN, IC2C.+IN, IC2D.+IN, JP4.2; no longer IC11A.+IN, IC11B.+IN, IC11C.+IN, IC11D.+IN, IC18A.+IN, IC18B.+IN, IC19A.+IN, IC19B.+IN, IC23A.+IN, JP1.13, JP5.8, JP6.6, R117.1, R123.1, U3.AGND, U3.DGND, U4.GND, U4.V-
- net INTEG_IN1: now also IC1A.OUT, JP3.2, R14.2; no longer IC18D.OUT, JP4.1, R118.2
- net INTEG_IN11: now also JP3.7, R10.1; no longer JP4.2, R145.1
- net INTEG_IN2: now also IC1C.OUT, JP3.6, R16.2; no longer IC19D.OUT, JP4.3, R124.2
- net INTEG_IN22: now also JP3.3, R8.1; no longer JP4.4, R3.1
- net N$36: now also R1.2
- net N$38: now also R2.2
- net N$42: now also R11.2, R12.2; no longer R32.2
- net VIN1: now also C5.1, IC2A.OUT, JP1.6, R9.2; no longer C37.1, IC23A.OUT, JP2.1, R141.2
- net VIN11: now also JP1.7; no longer JP2.2
- net VIN2: now also C4.1, IC2C.OUT, JP1.2, R7.2; no longer C1.1, IC1A.OUT, JP2.3, R1.2
- net VIN22: now also JP1.3, R28.1; no longer JP2.4, R62.1
Other:
- moved on the sheet: IC1A, IC3A, IC3B, IC3C, IC3D, R1, R26, R27, R28, R29, R3, R30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
